Commit message: description

File: src/agv_description/src/urdf/beam.xacro (robot description, xacro)
@@ -1,7 +1,4 @@
 <?xml version="1.0"?>
 <robot name="beam" xmlns:xacro="http://ros.org/wiki/xacro">
-    <material name="Gray">
-        <color rgba="0.7 0.7 0.7 1.0" />
-    </material>
     <xacro:macro name="box_inertia" params="m w h d">
         <inertial>

File: src/agv_description/src/urdf/caster.xacro (robot description, xacro)
@@ -1,14 +1,15 @@
 <?xml version="1.0"?>
-<robot name="caster" xmlns:xacro="http://ros.org/wiki/xacro">
-    <xacro:property name="caster_radius" value="0.035" />
-    <xacro:property name="caster_width" value="0.02" />
-    <xacro:macro name="cylinder_inertia" params="m r h">
-        <inertial>
-            <origin xyz="0 0 0" rpy="${pi/2} 0 0" />
-            <mass value="${m}" />
-            <inertia ixx="${(m/12) * (3*r*r + h*h)}" ixy="0" ixz="0" iyy="${(m/12) * (3*r*r + h*h)}" iyz="0" izz="${(m/2) * (r*r)}" />
-        </inertial>
-    </xacro:macro>
-    <xacro:macro name="sphere_inertia" params="m r">
+<robot name="caster"
+  xmlns:xacro="http://ros.org/wiki/xacro">
+  <xacro:property name="caster_radius" value="0.035" />
+  <xacro:property name="caster_width" value="0.02" />
+  <xacro:macro name="cylinder_inertia" params="m r h">
+    <inertial>
+      <origin xyz="0 0 0" rpy="${pi/2} 0 0" />
+      <mass value="${m}" />
+      <inertia ixx="${(m/12) * (3*r*r + h*h)}" ixy="0" ixz="0" iyy="${(m/12) * (3*r*r + h*h)}" iyz="0" izz="${(m/2) * (r*r)}" />
+    </inertial>
+  </xacro:macro>
+  <xacro:macro name="sphere_inertia" params="m r">
     <inertial>
       <mass value="${m}"/>
@@ -16,28 +17,28 @@
     </inertial>
   </xacro:macro>
-    <xacro:macro name="caster" params="parent prefix ztotal x y z">
-        <link name="${prefix}_link">
-            <visual>
-              <origin xyz="0 0 0" rpy="${pi/2} 0 0" />
-              <geometry>
-                <sphere radius="${caster_radius}" />
-              </geometry>
-              <material name="Black"/>
-            </visual>
-            <collision>
-              <origin xyz="0 0 0" rpy="${pi/2} 0 0" />
-              <geometry>
-                <cylinder radius="${caster_radius}" length="${caster_width}" />
-              </geometry>
-            </collision>
-            <xacro:sphere_inertia m="0.5" r="${caster_radius}"/>
-          </link>
-          <joint name="${prefix}_joint" type="continuous">
-            <parent link="${parent}" />
-            <child link="${prefix}_link" />
-            <origin xyz="${x} ${y} ${-(ztotal-caster_radius)}" rpy="0 0 0" />
-            <axis xyz="0 1 0" />
-          </joint>
-    </xacro:macro>
-    <!-- <xacro:beam prefix="c1" parent="base_link" length="0.48" height="0.02" x="0" y="0" z="0" r="1" /> -->
+  <xacro:macro name="caster" params="parent prefix ztotal x y z">
+    <link name="${prefix}_link">
+      <visual>
+        <origin xyz="0 0 0" rpy="${pi/2} 0 0" />
+        <geometry>
+          <sphere radius="${caster_radius}" />
+        </geometry>
+        <material name="Black"/>
+      </visual>
+      <collision>
+        <origin xyz="0 0 0" rpy="${pi/2} 0 0" />
+        <geometry>
+          <cylinder radius="${caster_radius}" length="${caster_width}" />
+        </geometry>
+      </collision>
+      <xacro:sphere_inertia m="0.5" r="${caster_radius}"/>
+    </link>
+    <joint name="${prefix}_joint" type="fixed">
+      <parent link="${parent}" />
+      <child link="${prefix}_link" />
+      <origin xyz="${x} ${y} ${-(ztotal-caster_radius)+0.001}" rpy="0 0 0" />
+      <axis xyz="0 1 0" />
+    </joint>
+  </xacro:macro>
+  <!-- <xacro:beam prefix="c1" parent="base_link" length="0.48" height="0.02" x="0" y="0" z="0" r="1" /> -->
 </robot>

File: src/agv_description/src/urdf/driver_assembly.xacro (robot description, xacro)
@@ -16,9 +16,4 @@
       </inertial>
     </link>
-    <!-- <joint name="driver_base_joint" type="fixed">
-      <parent link="base_link" />
-      <child link="driver_base" />
-      <origin xyz="0 0 0" rpy="0 0 0" />
-    </joint> -->
     <xacro:beam prefix="d1" parent="driver_base" length="0.22" height="0.02" x="-0.1" y="0" z="0" r="1" />
     <xacro:beam prefix="d2" parent="driver_base" length="0.22" height="0.02" x="0.1" y="0" z="0" r="1" />

File: src/agv_description/src/urdf/main.xacro (robot description, xacro)
@@ -70,12 +70,12 @@
     <plugin name='diff_drive' filename='libgazebo_ros_diff_drive.so'>
       <ros>
-        <namespace>/demo</namespace>
+        <namespace>/</namespace>
       </ros>
       <!-- wheels -->
-      <left_joint>drivewhl_l_joint</left_joint>
-      <right_joint>drivewhl_r_joint</right_joint>
+      <left_joint>lwheel_joint</left_joint>
+      <right_joint>rwheel_joint</right_joint>
       <!-- kinematics -->
-      <wheel_separation>0.025</wheel_separation>
-      <wheel_diameter>0.2</wheel_diameter>
+      <wheel_separation>${2*wheel_yoff}</wheel_separation>
+      <wheel_diameter>${2*wheel_radius}</wheel_diameter>
       <!-- limits -->
       <max_wheel_torque>20</max_wheel_torque>

File: src/agv_description/src/urdf/sensors/kinect.xacro (robot description, xacro)
@@ -26,5 +26,5 @@
         </joint>
         <gazebo reference="camera_link">
-            <sensor name="depth_camera" type="depth">
+            <sensor name="kinect" type="depth">
                 <visualize>true</visualize>
                 <update_rate>30.0</update_rate>
@@ -37,6 +37,6 @@
                     </image>
                     <clip>
-                        <near>0.05</near>
-                        <far>3</far>
+                        <near>0.08</near>
+                        <far>10</far>
                     </clip>
                 </camera>
@@ -46,6 +46,6 @@
                     <updateRate>0.0</updateRate>
                     <frameName>camera_depth_frame</frameName>
-                    <pointCloudCutoff>0.5</pointCloudCutoff>
-                    <pointCloudCutoffMax>3.0</pointCloudCutoffMax>
+                    <pointCloudCutoff>0.8</pointCloudCutoff>
+                    <pointCloudCutoffMax>4.0</pointCloudCutoffMax>
                     <distortionK1>0</distortionK1>
                     <distortionK2>0</distortionK2>

File: src/agv_description/src/urdf/wheel.xacro (robot description, xacro)
@@ -1,4 +1,5 @@
 <?xml version="1.0"?>
-<robot name="wheel" xmlns:xacro="http://www.ros.org/wiki/xacro">
+<robot name="wheel"
+  xmlns:xacro="http://www.ros.org/wiki/xacro">
   <xacro:property name="wheel_radius" value="0.045" />
   <xacro:property name="wheel_width" value="0.04" />
@@ -30,6 +31,6 @@
       <parent link="base_link" />
       <child link="${prefix}_link" />
+      <axis rpy="0 0 0" xyz="0 1 0"/>
       <origin xyz="0 ${yoff} 0" rpy="0 0 0" />
-      <axis xyz="0 1 0" />
     </joint>
   </xacro:macro>
